File: hw/v0.2/BG95.kicad_sch (KiCad schematic)
At the start: 51 parts, among them J1 USB_C_Receptacle_USB2.0, J4 JAE_SIM_Card_SF72S006, Q2 BSS138, SW1 SW_Omron_B3FS, U1 BG95M3LA-64-SGNS, U12 D3V3XA4B10LP

Commit message: update the quecpython project
Parts:
- added TP1: TestPoint, TestPoint:TestPoint_Pad_D1.0mm, symbol Connector:TestPoint
Connections:
- net at U1.2 (ADC1): now also TP1.1
- no-connect marks 13 -> 12
Changed lines of the file:
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@@
   (no_connect (at 220.98 68.58))
   (no_connect (at 170.18 92.71))
-  (no_connect (at 220.98 102.87))
   (no_connect (at 220.98 105.41))
   (no_connect (at 170.18 88.9))
@@
   )
   (wire (pts (xy 68.58 142.24) (xy 68.58 162.56))
+    (stroke (width 0) (type default))
+  )
+  (wire (pts (xy 224.155 102.87) (xy 220.98 102.87))
     (stroke (width 0) (type default))
   )
@@
         )
       )
+    )
+  )
+  (symbol (lib_id "Connector:TestPoint") (at 224.155 102.87 270) (unit 1)
+    (in_bom yes) (on_board yes) (dnp no)
+    (property "Reference" "TP1" (at 227.965 102.87 90)
+      (effects (font (size 1.27 1.27)) (justify left))
+    )
+    (property "Value" "TestPoint" (at 229.235 104.14 90)
+      (effects (font (size 1.27 1.27)) (justify left) hide)
+    )
+    (property "Footprint" "TestPoint:TestPoint_Pad_D1.0mm" (at 224.155 107.95 0)
+      (effects (font (size 1.27 1.27)) hide)
+    )
+    (property "Datasheet" "~" (at 224.155 107.95 0)
+      (effects (font (size 1.27 1.27)) hide)
+    )
+    (pin "1")
+    (instances
+      (project "IOT"
+        (path "/a6ff655f-285e-495a-9f3d-0c2e60b8700b/1642d687-ae69-4219-9a88-a808b8a284e1"
+          (reference "TP1") (unit 1)
+        )
+      )
