File: hw/v0.2/IOT.kicad_pcb (KiCad board)
At the start: 4 copper layers, 26.4 x 50.8 mm, 110 parts, among them J1 USB_C_Receptacle_USB2.0, J2 Feather Interface, J3 Feather Interface, J4 JAE_SIM_Card_SF72S006, J5 S2B-PH-SM4-TB_LF__SN_, Q1 AO3401A, Q2 BSS138, SW1 SW_Omron_B3FS, U1 BG95M3LA-64-SGNS, U10 TXS0104EYZTR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

Commit message: update the quecpython project
Parts:
- added TP1: TestPoint, TestPoint:TestPoint_Pad_D1.0mm, B.Cu at (170.0, 92.4)
Connections:
- U1 pad 2: unconnected-(U1-ADC1-Pad2) -> Net-(U1-ADC1)
Routing:
- net Net-(U1-ADC1): track 0.00 -> 3.24 mm, vias 0 -> 1
- net /Interface/A0: track 13.9 -> 14.7 mm
Other:
- board text removed: "Build your next IoT project in python"
