File: hw/v0.2/Power.kicad_sch (KiCad schematic)
At the start: 34 parts, among them J5 S2B-PH-SM4-TB_LF__SN_, Q1 AO3401A, U13 TLV75533PDRV, U14 RT9526AGQW, U2 TPS63020DSJR, U8 XC6119C32A7R-G

Commit message: update the quecpython project
Other:
- moved on the sheet: C19, C20, C21, C28, C32, C40, C41, D6, D7, R11, R19, R9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
